File: Measurements.kicad_sch (KiCad schematic)
At the start: 4 parts

Commit message: Первая версия в производство
Parts:
- C3, C7: value C_Small -> 1u
- R4: value R_Small -> 200
Changed lines of the file:
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@@
       (effects (font (size 1.27 1.27)) (justify left))
     )
-    (property "Value" "R_Small" (id 1) (at 83.947 114.5539 0)
+    (property "Value" "200" (id 1) (at 83.947 114.5539 0)
       (effects (font (size 1.27 1.27)) (justify left))
     )
@@
       (effects (font (size 1.27 1.27)) (justify left))
     )
-    (property "Value" "C_Small" (id 1) (at 84.201 121.9262 0)
+    (property "Value" "1u" (id 1) (at 84.201 121.9262 0)
       (effects (font (size 1.27 1.27)) (justify left))
     )
@@
       (effects (font (size 1.27 1.27)) (justify left))
     )
-    (property "Value" "C_Small" (id 1) (at 60.325 109.2262 0)
+    (property "Value" "1u" (id 1) (at 60.325 109.2262 0)
       (effects (font (size 1.27 1.27)) (justify left))
     )
