File: Power.kicad_pcb (KiCad board)
At the start: 4 copper layers, 138.7 x 119.4 mm, 50 parts, among them J1 OUT-, J2 OUT+, J3 IN+, J4 IN-, J5 Conn_02x05_Odd_Even, U1 TMR_1-0511

Commit message: VER2.0
Parts:
- removed F1: Fuse, Fuse:Fuse_2512_6332Metric_Pad1.52x3.35mm_HandSolder
- added C24: 100u, Capacitor_4pin:C4AE, F.Cu at (161.8, 82.1)
- added C25: C_Small, Capacitor_SMD:C_1210_3225Metric_Pad1.33x2.70mm_HandSolder, F.Cu at (102.6, 63.8)
- added J6: L_IN, Connector Power:M5, F.Cu at (209.0, 37.6)
- added J7: L_OUT, Connector Power:M5, F.Cu at (186.7, 60.2)
- C10, C19, C20, C21, C22, C23: moved to F.Cu
- moved H4 206.1 mm to (220.7, 62.0)
- moved J3 85.1 mm to (209.6, 59.9)
- moved F2 75.7 mm to (201.7, 48.5)
- moved R3 75.5 mm to (145.0, 51.1), turned to 90 degrees
- moved R2 72.1 mm to (145.0, 59.7), turned to 90 degrees
- moved H1 64.6 mm to (220.7, 35.8)
- moved R4 63.9 mm to (140.5, 56.7), turned to 180 degrees
- moved C5 63.7 mm to (137.2, 47.5), turned to 90 degrees
- moved J4 61.1 mm to (161.3, 37.6)
- moved C4 60.3 mm to (137.2, 51.6), turned to 90 degrees
- moved C3 57.8 mm to (137.2, 55.6), turned to 90 degrees
- moved C22 50.1 mm to (132.1, 58.9), turned to 0 degrees
- moved D3 43.3 mm to (128.0, 52.1), turned to 180 degrees
- moved J1 36.8 mm to (186.4, 37.6)
- moved C9 36.5 mm to (119.4, 47.5), turned to 90 degrees
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Connections:
- F2 pad 1: /input current -> /IN+
- L1 pad 2: Net-(L1-Pad2) -> /OUT+
- R2 pad 1: /input current -> /IN+
Routing:
- net /input current: track 125.5 -> 0.00 mm, vias 2 -> 0
- net +5VP: track 29.8 -> 85.1 mm, vias 3 -> 0
- net /Current_measure: track 33.1 -> 82.8 mm
- net /Output_Voltage: track 24.6 -> 43.2 mm, vias 2 -> 3
- net /OUT+: track 8.38 -> 23.6 mm
- net GND: track 68.0 -> 53.0 mm, vias 7 -> 6
- net /IN+: track 0.00 -> 11.1 mm, vias 0 -> 1
- net /Input_Voltage: track 46.9 -> 55.5 mm, vias 2 -> 3
- net GNDPWR: track 35.1 -> 31.4 mm, vias 5 -> 6
- net +5V: track 69.1 -> 67.7 mm, vias 7 -> 4
- added copper zone on In2.Cu, net +5V
- added copper zone on F.Cu, net /IN+
- added copper zone on In1.Cu, net /IN+
- added copper zone on In1.Cu, net GND
- added copper zone on F.Cu, net GNDPWR
- removed copper zone on B.Cu, net +5V
- removed copper zone on In1.Cu, net +5V
- removed copper zone on B.Cu, net +5VP
- removed copper zone on B.Cu, net GND
- removed copper zone on In2.Cu, net GND
- removed copper zone on F.Cu, net Net-(L1-Pad2)
Other:
- board size 138.7 x 119.4 mm -> 192 x 109.2 mm

Commit message: Готовый вариант
Parts:
- removed C1: 100u, Capacitor_4pin:C4AE
- removed C10, C16, C18, C19, C9: 470p, Capacitor_SMD:C_0805_2012Metric_Pad1.18x1.45mm_HandSolder
- removed C11, C2, C22, C23: C_Small, Capacitor_SMD:C_0805_2012Metric_Pad1.18x1.45mm_HandSolder
- removed C12: 0.01u, Capacitor_SMD:C_0805_2012Metric_Pad1.18x1.45mm_HandSolder
- removed C13, C14, C15, C17, C4, C5, C6, C8: 0.1u, Capacitor_SMD:C_0805_2012Metric_Pad1.18x1.45mm_HandSolder
- removed C20, C25: C_Small, Capacitor_SMD:C_1210_3225Metric_Pad1.33x2.70mm_HandSolder
- removed D3, D5: HCPL788J, Package_SO:SOIC-16W_7.5x10.3mm_P1.27mm
- removed F2: Fuse, Fuse:Fuse_2920_7451Metric_Pad2.10x5.45mm_HandSolder
- removed H1, H2, H4: MountingHole, MountingHole:MountingHole_3.2mm_M3
- removed J7: L_OUT, Connector Power:M5
- removed R1: R_Small, Resistor_SMD:R_0805_2012Metric_Pad1.20x1.40mm_HandSolder
- removed R2, R3, R6, R7: R, Resistor_SMD:R_2512_6332Metric_Pad1.40x3.35mm_HandSolder
- removed R5, R9: 4.7k, Resistor_SMD:R_0805_2012Metric_Pad1.20x1.40mm_HandSolder
- removed R8: 39, Resistor_SMD:R_0805_2012Metric_Pad1.20x1.40mm_HandSolder
- removed U1: TMR_1-0511, Converter_DCDC:Converter_DCDC_TRACO_TMR-1-xxxx_Single_THT
- added F1: Fuse, Fuse:Fuse_2920_7451Metric_Pad2.10x5.45mm_HandSolder, F.Cu at (77.2, 59.2)
- added J10: Voltage_Measure, Connector_Molex:Molex_Micro-Fit_3.0_43045-0412_2x02_P3.00mm_Vertical, F.Cu at (179.3, 131.8)
- added J8: +5V, Connector_Molex:Molex_Micro-Fit_3.0_43045-0412_2x02_P3.00mm_Vertical, F.Cu at (204.2, 131.8)
- added J9: Current_Measure, Connector_Molex:Molex_Micro-Fit_3.0_43045-0412_2x02_P3.00mm_Vertical, F.Cu at (191.7, 131.8)
- C21: value C_Small -> 100u; footprint Capacitor_SMD:C_1210_3225Metric_Pad1.33x2.70mm_HandSolder -> Capacitor_4pin:C4AE
- C3: value 0.01u -> C_Small; moved to B.Cu
- C7: value 470p -> C_Small; moved to B.Cu
- D4: moved to B.Cu
- J1: value OUT- -> OUT+; footprint Connector Power:M5 -> Connector_Molex:Molex_Micro-Fit_3.0_43045-0412_2x02_P3.00mm_Vertical
- J2: value OUT+ -> OUT-; footprint Connector Power:M5 -> Connector_Molex:Molex_Micro-Fit_3.0_43045-0412_2x02_P3.00mm_Vertical
- J3: value IN+ -> L_OUT; footprint Connector Power:M5 -> Connector_Molex:Molex_Micro-Fit_3.0_43045-0812_2x04_P3.00mm_Vertical
- J4: value IN- -> L_IN; footprint Connector Power:M5 -> Connector_Molex:Molex_Micro-Fit_3.0_43045-0812_2x04_P3.00mm_Vertical
- J5: value Conn_02x05_Odd_Even -> IN+; footprint Connector_IDC:IDC-Header_2x05_P2.54mm_Vertical -> Connector_Molex:Molex_Micro-Fit_3.0_43045-0812_2x04_P3.00mm_Vertical
- J6: value L_IN -> IN-; footprint Connector Power:M5 -> Connector_Molex:Molex_Micro-Fit_3.0_43045-0812_2x04_P3.00mm_Vertical
- R4: value 39 -> R_Small; moved to B.Cu
- moved H3 179.4 mm to (216.2, 61.2)
- moved J5 109.3 mm to (196.4, 54.0), turned to 0 degrees
- moved J1 96.4 mm to (91.4, 54.0)
- moved C7 87.4 mm to (182.4, 105.4)
- moved C3 69.0 mm to (185.7, 104.6), turned to 180 degrees
- moved J4 65.5 mm to (218.5, 69.4), turned to -90 degrees
- moved R4 62.8 mm to (180.1, 105.4), turned to -90 degrees
- moved C21 59.5 mm to (116.3, 120.1), turned to 180 degrees
- moved J2 47.9 mm to (106.3, 54.0)
- moved J6 37.0 mm to (175.8, 54.0)
- moved C24 36.0 mm to (192.1, 62.5)
- moved L1 30.8 mm to (69.6, 71.1)
- moved D1 30.2 mm to (154.2, 69.5)
- moved D2 30.0 mm to (81.0, 69.6)
- moved J3 29.4 mm to (218.5, 88.0), turned to -90 degrees
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Connections:
- net /output current renamed LPSR_OUT
- C21 pad 1: +5VP -> Net-(C21-Pad1)
- C24 pad 1: /IN+ -> Voltage_IN
- C3 pad 1: Net-(C3-Pad1) -> +5V
- C3 pad 2: Net-(C3-Pad2) -> GND
- C7 pad 1: Net-(C7-Pad1) -> Current_Measure
- D1 pad 3: Net-(C1-Pad1) -> Net-(C21-Pad1)
- D2 pad 2: Net-(C1-Pad1) -> Net-(C21-Pad1)
- D4 pad 1: /input current -> LPSR_IN
- D4 pad 2: /input current -> LPSR_IN
- D4 pad 3: /input current -> LPSR_IN
- D4 pad 4: /input current -> LPSR_IN
- J1 pad 1: GNDPWR -> Voltage_OUT
- J2 pad 1: /OUT+ -> GNDPWR
- J3 pad 1: Net-(J3-Pad1) -> LPSR_IN
- J4 pad 1: GNDPWR -> Voltage_IN
- J5 pad 1: /Output_Voltage -> Voltage_IN
- J5 pad 2: GND -> Voltage_IN
- J5 pad 3: /Input_Voltage -> Voltage_IN
- J5 pad 4: GND -> Voltage_IN
- J5 pad 5: +5V -> Voltage_IN
- J5 pad 6: GND -> Voltage_IN
- J5 pad 7: +5V -> Voltage_IN
- J5 pad 8: GND -> Voltage_IN
- J6 pad 1: /IN+ -> GNDPWR
- L1 pad 2: /OUT+ -> Net-(F1-Pad1)
- R4 pad 1: Net-(R2-Pad2) -> Net-(D4-Pad11)
- R4 pad 2: Net-(C3-Pad1) -> Current_Measure
Routing:
- net +5VP: track 85.1 -> 0.00 mm
- net /Current_measure: track 82.8 -> 0.00 mm
- net /Input_Voltage: track 55.5 -> 0.00 mm, vias 3 -> 0
- net Voltage_OUT: track 0.00 -> 44.5 mm
- net /Output_Voltage: track 43.2 -> 0.00 mm, vias 3 -> 0
- net Voltage_IN: track 0.00 -> 33.8 mm
- net GNDPWR: track 31.4 -> 0.00 mm, vias 6 -> 0
- net Current_Measure: track 0.00 -> 30.3 mm, vias 0 -> 1
- net +5V: track 67.7 -> 42.9 mm, vias 4 -> 1
- net /OUT+: track 23.6 -> 0.00 mm
- net GND: track 53.0 -> 32.8 mm, vias 6 -> 1
- net /IN+: track 11.1 -> 0.00 mm, vias 1 -> 0
- net Net-(C7-Pad1): track 10.7 -> 0.00 mm
- net Net-(C16-Pad1): track 10.7 -> 0.00 mm
- net Net-(C12-Pad1): track 6.87 -> 0.00 mm
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- added copper zone on F.Cu, net LPSR_IN
- added copper zone on F.Cu, net Net-(C21-Pad1)
- added copper zone on F.Cu, net Net-(F1-Pad1)
- added copper zone on F.Cu, net Voltage_IN
- added copper zone on In2.Cu, net Voltage_IN
- added copper zone on F.Cu, net Voltage_OUT
- added copper zone on In2.Cu, net Voltage_OUT
- removed copper zone on In2.Cu, net +5V
- removed copper zone on F.Cu, net /IN+
- removed copper zone on In1.Cu, net /IN+
- removed copper zone on F.Cu, net /OUT+
- removed copper zone on F.Cu, net /input current
- removed copper zone on F.Cu, net GNDPWR
- removed copper zone on F.Cu, net Net-(C1-Pad1)
- removed copper zone on F.Cu, net Net-(J3-Pad1)
Other:
- board size 192 x 109.2 mm -> 160.3 x 92.2 mm
- board text added: "+"
- board text added: "-"
- board text added: "5V Supply"
- board text added: "Current Measure"
- board text added: "GND"
- board text added: "I OUT"
- board text added: "Input Voltage"
- board text added: "J1"
- board text added: "J2"
- board text added: "J5"
- board text added: "J6"
- board text added: "L IN"
- board text added: "L OUT"
- board text added: "Output Voltage"
- board text added: "V IN"
- board text added: "V OUT"
- board text added: "Voltage Measure"

Commit message: Первая версия в производство
Parts:
- F1: footprint Fuse:Fuse_2920_7451Metric_Pad2.10x5.45mm_HandSolder -> Fuse:Fuse_2512_6332Metric_Pad1.52x3.35mm_HandSolder
- moved J5 25.0 mm to (221.4, 54.0)
- moved H3 23.8 mm to (238.9, 54.4)
- moved J6 10.0 mm to (165.8, 54.0)
Other:
- board size 160.3 x 92.2 mm -> 179.1 x 92.2 mm
