File: Power.kicad_sch (KiCad schematic)
At the start: 50 parts, among them J1 OUT-, J2 OUT+, J3 IN+, J4 IN-, J5 Conn_02x05_Odd_Even

Commit message: VER1.0
Parts:
- removed F1: Fuse, Fuse:Fuse_2512_6332Metric_Pad1.52x3.35mm_HandSolder, symbol Device:Fuse
- added C24: 100u, Capacitor_4pin:C4AE, symbol Device:C
- added C25: C_Small, Capacitor_SMD:C_1210_3225Metric_Pad1.33x2.70mm_HandSolder, symbol Device:C_Small
- added J6: L_IN, Connector Power:M5, symbol Connector_Generic:Conn_01x01
- added J7: L_OUT, Connector Power:M5, symbol Connector_Generic:Conn_01x01
- gave numbers to parts that had none: 1
Connections:
- net +5VP: now also C25.1
- net GNDPWR: now also C24.2, C25.2
- net OUT+: now also L1.2
- net input current: now also J7.1 (Pin_1); no longer F2.1, R2.1
- new net IN+: C24.1, F2.1, J6.1 (Pin_1), R2.1
Other:
- moved on the sheet: H1, H2, H3, H4

Commit message: Готовый вариант
Parts:
- removed C1, C24: 100u, Capacitor_4pin:C4AE, symbol Device:C
- removed C10, C16, C18, C19, C7, C9: 470p, Capacitor_SMD:C_0805_2012Metric_Pad1.18x1.45mm_HandSolder, symbol Device:C_Small
- removed C11, C2, C22, C23: C_Small, Capacitor_SMD:C_0805_2012Metric_Pad1.18x1.45mm_HandSolder, symbol Device:C_Small
- removed C12, C3: 0.01u, Capacitor_SMD:C_0805_2012Metric_Pad1.18x1.45mm_HandSolder, symbol Device:C_Small
- removed C13, C14, C15, C17, C4, C5, C6, C8: 0.1u, Capacitor_SMD:C_0805_2012Metric_Pad1.18x1.45mm_HandSolder, symbol Device:C_Small
- removed C20, C21, C25: C_Small, Capacitor_SMD:C_1210_3225Metric_Pad1.33x2.70mm_HandSolder, symbol Device:C_Small
- removed D1, D2: SKM100GB12T4, IGBT_Modul:SEMITRANS_2, symbol IGBT_Modul:SKM100GB12T4
- removed D3, D5: HCPL788J, Package_SO:SOIC-16W_7.5x10.3mm_P1.27mm, symbol HCPL:HCPL788J
- removed D4: LPSR_50-NP, LPSR:LPSR_50, symbol LPSR:LPSR_50-NP
- removed F2: Fuse, Fuse:Fuse_2920_7451Metric_Pad2.10x5.45mm_HandSolder, symbol Device:Fuse
- removed H1, H2, H3, H4: MountingHole, MountingHole:MountingHole_3.2mm_M3, symbol Mechanical:MountingHole
- removed J1: OUT-, Connector Power:M5, symbol Connector_Generic:Conn_01x01
- removed J2: OUT+, Connector Power:M5, symbol Connector_Generic:Conn_01x01
- removed J3: IN+, Connector Power:M5, symbol Connector_Generic:Conn_01x01
- removed J4: IN-, Connector Power:M5, symbol Connector_Generic:Conn_01x01
- removed J5: Conn_02x05_Odd_Even, Connector_IDC:IDC-Header_2x05_P2.54mm_Vertical, symbol Connector_Generic:Conn_02x05_Odd_Even
- removed J6: L_IN, Connector Power:M5, symbol Connector_Generic:Conn_01x01
- removed J7: L_OUT, Connector Power:M5, symbol Connector_Generic:Conn_01x01
- removed L1: L_Small, Inductor_My:Wurth, symbol Device:L_Small
- removed R1: R_Small, Resistor_SMD:R_0805_2012Metric_Pad1.20x1.40mm_HandSolder, symbol Device:R_Small
- removed R2, R3, R6, R7: R, Resistor_SMD:R_2512_6332Metric_Pad1.40x3.35mm_HandSolder, symbol Device:R
- removed R4, R8: 39, Resistor_SMD:R_0805_2012Metric_Pad1.20x1.40mm_HandSolder, symbol Device:R_Small
- removed R5, R9: 4.7k, Resistor_SMD:R_0805_2012Metric_Pad1.20x1.40mm_HandSolder, symbol Device:R_Small
- removed U1: TMR_1-0511, Converter_DCDC:Converter_DCDC_TRACO_TMR-1-xxxx_Single_THT, symbol Regulator_Switching:TMR_1-0511
Connections:
- no-connect marks 7 -> 0
Other:
- added sheet Connector (Connector.kicad_sch)
- added sheet Measurements (Measurements.kicad_sch)
- added sheet PowerIGBT (PowerIGBT.kicad_sch)
