File: PowerIGBT.kicad_sch (KiCad schematic)
At the start: 12 parts, among them J1 OUT+, J2 OUT-, J3 L_OUT, J4 L_IN, J5 IN+, J6 IN-

Commit message: Поменял предохранитель
Parts:
- F1: footprint Fuse:Fuse_2920_7451Metric_Pad2.10x5.45mm_HandSolder -> Fuse:Fuse_2512_6332Metric_Pad1.52x3.35mm_HandSolder
Changed lines of the file:
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@@
       (effects (font (size 1.27 1.27)) (justify left))
     )
-    (property "Footprint" "Fuse:Fuse_2920_7451Metric_Pad2.10x5.45mm_HandSolder" (id 2) (at 151.892 85.598 90)
+    (property "Footprint" "Fuse:Fuse_2512_6332Metric_Pad1.52x3.35mm_HandSolder" (id 2) (at 151.892 85.598 90)
       (effects (font (size 1.27 1.27)) hide)
     )

Commit message: Первая версия в производство
Parts:
- F1: value Fuse -> 0679L9200-01
Changed lines of the file:
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@@
     (in_bom yes) (on_board yes)
     (property "Reference" "L1" (id 0) (at 142.24 81.788 90))
-    (property "Value" "L_Small" (id 1) (at 142.24 85.598 90))
+    (property "Value" "L_Small" (id 1) (at 142.24 85.598 90)
+      (effects (font (size 1.27 1.27)) hide)
+    )
     (property "Footprint" "Inductor_My:Wurth" (id 2) (at 142.24 83.82 0)
       (effects (font (size 1.27 1.27)) hide)
@@
       (effects (font (size 1.27 1.27)) (justify left))
     )
-    (property "Value" "Fuse" (id 1) (at 154.178 85.852 90)
+    (property "Value" "0679L9200-01" (id 1) (at 159.258 86.106 90)
       (effects (font (size 1.27 1.27)) (justify left))
     )
